Commit message: 修改urdf

File: panda_description/urdf/panda.urdf (robot description, URDF)
Before this commit: robot panda, 12 links, 11 joints
Links:
- removed link panda_link0
- added link link0; collision mesh filename=package://panda_description/meshes/collision/link0.stl; visual mesh filename=package://panda_description/meshes/visual/link0.dae
- added link world
Joints:
- added joint base_joint: type fixed, parent world, child link0
- joint panda_joint1: parent panda_link0 -> link0

Commit message: 完成moveit和mujoco配置,moveit2正常控制

File: panda_description/urdf/panda.urdf (robot description, URDF)
Before this commit: robot panda, 13 links, 12 joints
Links:
- removed link link0
- added link panda_link0; collision mesh filename=package://panda_description/meshes/collision/link0.stl; visual mesh filename=package://panda_description/meshes/visual/link0.dae
Joints:
- joint base_joint: child link0 -> panda_link0
- joint panda_joint1: parent link0 -> panda_link0
